File: neo60core_rp2040.kicad_pcb (KiCad board)
At the start: 2 copper layers, 284.8 x 94.3 mm, 178 parts, among them J1 Conn_01x05, U1 RP2040, U2 XC6206PxxxMR, U3 W25Q128JVS, Y1 YSX321SL

Commit message: V1.1
Parts:
- C14, C15: value 33p -> 15p
- R4: value 100R -> 1K
- Y1: value YSX321SL -> ABM8-272-T3
- turned D1 to 90 degrees
Connections:
- D1 pad 1: Net-(D1-K) -> Row0
- D1 pad 2: Row0 -> Net-(D1-A)
- MX1 pad 2: Net-(D1-K) -> Net-(D1-A)
Routing:
- net Net-(D1-K): track 5.05 -> 0.00 mm
- net Net-(D1-A): track 0.00 -> 5.05 mm
Changed lines of the file:
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@@
 	(net 103 "unconnected-(U1-GPIO29_ADC3-Pad41)")
 	(net 104 "unconnected-(U1-GPIO28_ADC2-Pad40)")
-	(net 105 "Net-(D1-K)")
+	(net 105 "Net-(D1-A)")
 	(net 106 "Net-(D62-A)")
 	(net 107 "DP")
@@
 			(layers "*.Cu" "*.Mask")
 			(remove_unused_layers no)
-			(net 105 "Net-(D1-K)")
+			(net 105 "Net-(D1-A)")
 			(pinfunction "2")
 			(pintype "passive")
@@
 			)
 		)
-		(property "Value" "YSX321SL"
+		(property "Value" "ABM8-272-T3"
 			(at 0 -2.450001 -90)
 			(layer "B.Fab")
@@
 			)
 		)
-		(property "Value" "33p"
+		(property "Value" "15p"
 			(at 0 -1.679999 -90)
 			(layer "B.Fab")
@@
 			)
 		)
+		(sheetname "Root")
+		(sheetfile "neo60core_rp2040.kicad_sch")
 		(attr smd)
 		(fp_line
@@
 			)
 		)
-		(property "Value" "33p"
+		(property "Value" "15p"
 			(at 0 -1.679999 90)
 			(layer "B.Fab")
@@
 	(footprint "ScottoKeebs_Components:Diode_SOD-123_noref"
 		(layer "B.Cu")
-		(at 43.6 34.71875 -90)
+		(at 43.6 34.71875 90)
 		(descr "SOD-123")
 		(tags "SOD-123")
@@
 		)
 		(property "Value" "D_Small"
-			(at 0 -2.1 -90)
+			(at 0 -2.1 270)
 			(layer "B.Fab")
 			(effects
@@
 		)
 		(property "Footprint" "ScottoKeebs_Components:Diode_SOD-123_noref"
-			(at 0 0 90)
+			(at 0 0 -90)
 			(unlocked yes)
 			(layer "B.Fab")
@@
 		)
 		(property "Datasheet" ""
-			(at 0 0 90)
+			(at 0 0 -90)
 			(unlocked yes)
 			(layer "B.Fab")
@@
 		)
 		(property "Description" "Diode, small symbol"
-			(at 0 0 90)
+			(at 0 0 -90)
 			(unlocked yes)
 			(layer "B.Fab")
@@
 		)
 		(property "Sim.Device" "D"
-			(at 0 0 90)
+			(at 0 0 -90)
 			(unlocked yes)
 			(layer "B.Fab")
@@
 		)
 		(property "Sim.Pins" "1=K 2=A"
-			(at 0 0 90)
+			(at 0 0 -90)
 			(unlocked yes)
 			(layer "B.Fab")
@@
 		(attr smd)
 		(fp_line
-			(start -0.35 0.55)
-			(end -0.35 0)
+			(start -0.35 -0.55)
+			(end -0.349999 0)
 			(stroke
 				(width 0.15)
@@
 		)
 		(fp_line
-			(start 0.25 0.4)
-			(end -0.35 0)
+			(start 0.25 -0.4)
+			(end 0.25 0.4)
 			(stroke
 				(width 0.15)
@@
 		)
 		(fp_line
-			(start -0.35 0)
-			(end -0.75 0)
+			(start 0.75 0)
+			(end 0.25 0)
 			(stroke
 				(width 0.15)
@@
 		)
 		(fp_line
-			(start -0.35 0)
+			(start -0.349999 0)
 			(end 0.25 -0.4)
 			(stroke
@@
 		)
 		(fp_line
-			(start 0.75 0)
-			(end 0.25 0)
+			(start -0.349999 0)
+			(end -0.75 0)
 			(stroke
 				(width 0.15)
@@
 		)
 		(fp_line
-			(start 0.25 -0.4)
-			(end 0.25 0.4)
+			(start 0.25 0.4)
+			(end -0.349999 0)
 			(stroke
 				(width 0.15)
@@
 		)
 		(fp_line
-			(start -0.35 -0.55)
-			(end -0.35 0)
+			(start -0.35 0.55)
+			(end -0.349999 0)
 			(stroke
 				(width 0.15)
@@
 		)
 		(fp_line
-			(start 2.35 1.15)
-			(end -2.35 1.15)
+			(start 2.35 -1.15)
+			(end 2.35 1.15)
 			(stroke
 				(width 0.05)
@@
 		(fp_line
 			(start -2.35 -1.15)
-			(end -2.35 1.15)
+			(end 2.35 -1.15)
 			(stroke
 				(width 0.05)
@@
 		(fp_line
 			(start -2.35 -1.15)
-			(end 2.35 -1.15)
+			(end -2.35 1.15)
 			(stroke
 				(width 0.05)
@@
 		)
 		(fp_line
-			(start 2.35 -1.15)
-			(end 2.35 1.15)
+			(start 2.35 1.15)
+			(end -2.35 1.15)
 			(stroke
 				(width 0.05)
@@
 		)
 		(fp_line
-			(start -1.4 0.9)
-			(end -1.4 -0.9)
+			(start 1.4 -0.900001)
+			(end 1.4 0.900001)
 			(stroke
 				(width 0.1)
@@
 		)
 		(fp_line
-			(start 1.4 0.9)
-			(end -1.4 0.9)
+			(start -1.4 -0.900001)
+			(end 1.4 -0.900001)
 			(stroke
 				(width 0.1)
@@
 		)
 		(fp_line
-			(start -0.35 0.55)
-			(end -0.35 0)
+			(start -0.35 -0.55)
+			(end -0.349999 0)
 			(stroke
 				(width 0.1)
@@
 		)
 		(fp_line
-			(start 0.25 0.4)
-			(end -0.35 0)
+			(start 0.25 -0.4)
+			(end 0.25 0.4)
 			(stroke
 				(width 0.1)
@@
 		)
 		(fp_line
-			(start -0.35 0)
-			(end -0.75 0)
+			(start 0.75 0)
+			(end 0.25 0)
 			(stroke
 				(width 0.1)
@@
 		)
 		(fp_line
-			(start -0.35 0)
+			(start -0.349999 0)
 			(end 0.25 -0.4)
 			(stroke
@@
 		)
 		(fp_line
-			(start 0.75 0)
-			(end 0.25 0)
+			(start -0.349999 0)
+			(end -0.75 0)
 			(stroke
 				(width 0.1)
@@
 		)
 		(fp_line
-			(start 0.25 -0.4)
-			(end 0.25 0.4)
+			(start 0.25 0.4)
+			(end -0.349999 0)
 			(stroke
 				(width 0.1)
@@
 		)
 		(fp_line
-			(start -0.35 -0.55)
-			(end -0.35 0)
+			(start -0.35 0.55)
+			(end -0.349999 0)
 			(stroke
 				(width 0.1)
@@
 		)
 		(fp_line
-			(start -1.4 -0.9)
-			(end 1.4 -0.9)
+			(start 1.4 0.900001)
+			(end -1.4 0.900001)
 			(stroke
 				(width 0.1)
@@
 		)
 		(fp_line
-			(start 1.4 -0.9)
-			(end 1.4 0.9)
+			(start -1.4 0.900001)
+			(end -1.4 -0.900001)
 			(stroke
 				(width 0.1)
@@
 		)
 		(fp_text user "${REFERENCE}"
-			(at 0 2 -90)
+			(at 0 2.000001 270)
 			(layer "B.Fab")
 			(effects
@@
 		)
 		(pad "1" smd roundrect
-			(at -1.65 0 270)
+			(at -1.65 0 90)
 			(size 0.9 1.2)
 			(layers "B.Cu" "B.Paste" "B.Mask")
 			(roundrect_rratio 0.25)
-			(net 105 "Net-(D1-K)")
+			(net 7 "Row0")
 			(pinfunction "K")
 			(pintype "passive")
 		)
 		(pad "2" smd roundrect
-			(at 1.65 0 270)
+			(at 1.65 0 90)
 			(size 0.9 1.2)
 			(layers "B.Cu" "B.Paste" "B.Mask")
 			(roundrect_rratio 0.25)
-			(net 7 "Row0")
+			(net 105 "Net-(D1-A)")
 			(pinfunction "A")
 			(pintype "passive")
@@
 			)
 		)
-		(property "Value" "100R"
+		(property "Value" "1K"
 			(at 0 -1.65 -90)
 			(layer "B.Fab")
