File: neo60core_rp2040.kicad_sch (KiCad schematic)
At the start: 178 parts, among them J1 Conn_01x05, U1 RP2040, U2 XC6206PxxxMR, U3 W25Q128JVS, Y1 YSX321SL

Commit message: V1.1
Parts:
- C14, C15: value 33p -> 15p
- R4: value 100R -> 1K
- Y1: value YSX321SL -> ABM8-272-T3
Changed lines of the file:
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@@
 			)
 		)
-		(property "Value" "33p"
+		(property "Value" "15p"
 			(at 30.4863 138.43 90)
 			(effects
@@
 			)
 		)
-		(property "Value" "YSX321SL"
+		(property "Value" "ABM8-272-T3"
 			(at 40.64 129.032 90)
 			(effects
@@
 			)
 		)
-		(property "Value" "100R"
+		(property "Value" "1K"
 			(at 53.34 139.7 90)
 			(effects
@@
 			)
 		)
-		(property "Value" "33p"
+		(property "Value" "15p"
 			(at 30.4863 127 90)
 			(effects
